File: Eagle/SmartVision/SmartVision.sch (EAGLE design)
At the start: 52 parts, among them U1 SMALL_MAVRIC_IMU_MPU-9250, Y1 SMALL_MAVRIC_ABM10

Commit message: Fix supply and boot problem
Parts:
- added U$51: 1K, small_mavric:SMALL_MAVRIC_RESISTOR_R0402
Connections:
- removed net +3V: U$2.OUT, U$6.2
- removed net +3V3: U$1.VBAT, U$1.VDD1, U$1.VDD2, U$1.VDD3, U$1.VDD4, U$1.VDD5, U$1.VDD6, U$1.VDDA, U$1.VREF+, U$11.P10, U$11.P16, U$13.1, U$14.2, U$15.1, U$16.1, U$17.1, U$18.1, U$19.1, U$20.1, U$28.1, U$31.P1, U$34.1, U$38.2, U$39.1, U$48.1, U$49.1, U$50.1, U1.CSN, U1.REGOUT, U1.RESV(VDDIO), U1.VDD, U1.VDDIO
- removed net +3VANA: U$10.2, U$7.OUT
- new net VCC: U$1.VBAT, U$1.VDD1, U$1.VDD2, U$1.VDD3, U$1.VDD4, U$1.VDD5, U$1.VDD6, U$11.P10, U$13.1, U$14.2, U$15.1, U$16.1, U$17.1, U$18.1, U$19.1, U$2.OUT, U$20.1, U$31.P1, U$34.1, U$38.2, U$49.1, U$50.1, U$6.2, U1.CSN, U1.REGOUT, U1.RESV(VDDIO), U1.VDDIO
- new net VCC_ANA: U$1.VDDA, U$1.VREF+, U$10.2, U$11.P16, U$28.1, U$39.1, U$48.1, U$7.OUT, U1.VDD
- net GND: now also U$51.1
- net N$21: now also U$51.2
- net N$22: now also U$1.(BOOT1)_PB2; no longer U$1.PB2
Other:
- moved on the sheet: U$32

Commit message: Routing mostly complete !
Parts:
- added U$52: CON_2.54MM_16PINS_STACKABLE, STM32F4:CON_2.54MM_16PINS_STACKABLE
Connections:
- new net CAN2_RX: U$1.PB12, U$52.P15
- new net CAN2_TX: U$1.PB13, U$52.P16
- new net UART4_RX: U$1.PA1, U$52.P10
- new net UART4_TX: U$1.PA0, U$52.P9
- net GND: now also U$52.P1
- net I2C_SCL: now also U$52.P13
- net I2C_SDA: now also U$52.P14
Changed lines of the file:
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@@
 <setting verticaltext="up"/>
 </settings>
-<grid distance="0.1" unitdist="inch" unit="inch" style="lines" multiple="1" display="no" altdistance="0.01" altunitdist="inch" altunit="inch"/>
+<grid distance="0.1" unitdist="inch" unit="inch" style="lines" multiple="1" display="yes" altdistance="0.01" altunitdist="inch" altunit="inch"/>
 <layers>
 <layer number="1" name="Top" color="4" fill="1" visible="no" active="no"/>
@@
 <part name="P+8" library="supply1" deviceset="VCC" device=""/>
 <part name="P+9" library="supply1" deviceset="VCC" device=""/>
+<part name="U$52" library="STM32F4" deviceset="CON_2.54MM_16PINS_STACKABLE" device=""/>
+<part name="GND21" library="supply1" deviceset="GND" device=""/>
 </parts>
 <sheets>
@@
 </segment>
 </net>
+<net name="CAN2_RX" class="0">
+<segment>
+<pinref part="U$1" gate="G$1" pin="PB12"/>
+<wire x1="53.34" y1="-38.1" x2="73.66" y2="-38.1" width="0.1524" layer="91"/>
+<label x="66.04" y="-38.1" size="1.778" layer="95"/>
+</segment>
+</net>
+<net name="CAN2_TX" class="0">
+<segment>
+<pinref part="U$1" gate="G$1" pin="PB13"/>
+<wire x1="53.34" y1="-40.64" x2="73.66" y2="-40.64" width="0.1524" layer="91"/>
+<label x="66.04" y="-40.64" size="1.778" layer="95"/>
+</segment>
+</net>
+<net name="UART4_TX" class="0">
+<segment>
+<pinref part="U$1" gate="G$1" pin="PA0"/>
+<wire x1="53.34" y1="38.1" x2="73.66" y2="38.1" width="0.1524" layer="91"/>
+<label x="66.04" y="38.1" size="1.778" layer="95"/>
+</segment>
+</net>
+<net name="UART4_RX" class="0">
+<segment>
+<pinref part="U$1" gate="G$1" pin="PA1"/>
+<wire x1="53.34" y1="35.56" x2="73.66" y2="35.56" width="0.1524" layer="91"/>
+<label x="66.04" y="35.56" size="1.778" layer="95"/>
+</segment>
+</net>
 </nets>
 </sheet>
@@
 <instance part="P+6" gate="VCC" x="-71.12" y="-73.66"/>
 <instance part="P+7" gate="VCC" x="38.1" y="-50.8"/>
+<instance part="U$52" gate="G$1" x="96.52" y="10.16"/>
+<instance part="GND21" gate="1" x="96.52" y="-7.62"/>
 </instances>
 <busses>
@@
 <wire x1="30.48" y1="-86.36" x2="30.48" y2="-88.9" width="0.1524" layer="91"/>
 </segment>
+<segment>
+<pinref part="U$52" gate="G$1" pin="P1"/>
+<pinref part="GND21" gate="1" pin="GND"/>
+</segment>
 </net>
 <net name="USB_ID" class="0">
@@
 <junction x="-76.2" y="-68.58"/>
 </segment>
+<segment>
+<pinref part="U$52" gate="G$1" pin="P13"/>
+<wire x1="111.76" y1="17.78" x2="111.76" y2="38.1" width="0.1524" layer="91"/>
+<label x="111.76" y="30.48" size="1.778" layer="95" rot="R90"/>
+</segment>
 </net>
 <net name="I2C_SDA" class="0">
@@
 <junction x="38.1" y="-68.58"/>
 </segment>
+<segment>
+<pinref part="U$52" gate="G$1" pin="P14"/>
+<wire x1="106.68" y1="17.78" x2="106.68" y2="38.1" width="0.1524" layer="91"/>
+<label x="106.68" y="30.48" size="1.778" layer="95" rot="R90"/>
+</segment>
 </net>
 <net name="VCC" class="0">
@@
 </segment>
 </net>
+<net name="UART4_TX" class="0">
+<segment>
+<pinref part="U$52" gate="G$1" pin="P9"/>
+<wire x1="132.08" y1="17.78" x2="132.08" y2="38.1" width="0.1524" layer="91"/>
+<label x="132.08" y="30.48" size="1.778" layer="95" rot="R90"/>
+</segment>
+</net>
+<net name="UART4_RX" class="0">
+<segment>
+<pinref part="U$52" gate="G$1" pin="P10"/>
+<wire x1="127" y1="17.78" x2="127" y2="38.1" width="0.1524" layer="91"/>
+<label x="127" y="30.48" size="1.778" layer="95" rot="R90"/>
+</segment>
+</net>
+<net name="CAN2_RX" class="0">
+<segment>
+<pinref part="U$52" gate="G$1" pin="P15"/>
+<wire x1="101.6" y1="17.78" x2="101.6" y2="38.1" width="0.1524" layer="91"/>
+<label x="101.6" y="30.48" size="1.778" layer="95" rot="R90"/>
+</segment>
+</net>
+<net name="CAN2_TX" class="0">
+<segment>
+<pinref part="U$52" gate="G$1" pin="P16"/>
+<wire x1="96.52" y1="17.78" x2="96.52" y2="38.1" width="0.1524" layer="91"/>
+<label x="96.52" y="30.48" size="1.778" layer="95" rot="R90"/>
+</segment>
+</net>

Commit message: Routing finish
Routing without autorouter.
Need optimisation, symbol, value, …
Parts:
- added U$53: CON_1.25MM_4PINS, STM32F4:CON_1.25MM_4PINS
- added U$54: CON_2.54MM_2PINS_STACKABLE, STM32F4:CON_2.54MM_2PINS_STACKABLE
- added U$55, U$56, U$57, U$61: DIODE_SCHOTTKY, STM32F4:DIODE_SCHOTTKY
- added U$58, U$59, U$62: 28, small_mavric:SMALL_MAVRIC_RESISTOR_R0402
- added U$60: 12.5, small_mavric:SMALL_MAVRIC_RESISTOR_R0402
- U$10, U$34, U$5, U$6, U$9: device small_mavric:SMALL_MAVRIC_CAPACITOR_C0805 -> small_mavric:SMALL_MAVRIC_CAPACITOR_C0603
- U$12, U$14, U$25, U$26, U$27, U$38: device small_mavric:SMALL_MAVRIC_RESISTOR_R0603 -> small_mavric:SMALL_MAVRIC_RESISTOR_R0402
- U$13, U$15, U$16, U$17, U$18, U$19, U$20, U$21, U$22, U$28, U$3, U$30, U$39, U$48, U$49, U$50, U$8: device small_mavric:SMALL_MAVRIC_CAPACITOR_C0603 -> small_mavric:SMALL_MAVRIC_CAPACITOR_C0402
- U$44, U$45, U$46, U$47: value 100 -> 402; device small_mavric:SMALL_MAVRIC_RESISTOR_R0603 -> small_mavric:SMALL_MAVRIC_RESISTOR_R0402
- U$52: value CON_2.54MM_16PINS_STACKABLE -> CON_2.54MM_18PINS_STACKABLE; device STM32F4:CON_2.54MM_16PINS_STACKABLE -> STM32F4:CON_2.54MM_18PINS_STACKABLE
Connections:
- new net N$24: U$61.P2, U$62.1
- new net N$27: U$55.P2, U$58.1
- new net N$28: U$56.P2, U$59.1
- new net N$29: U$57.P2, U$60.1
- new net VBAT_C: U$53.P1, U$55.P1
- new net VBAT_P: U$54.P1, U$56.P1
- new net VBAT_S: U$52.P1, U$61.P1
- net CAN2_RX: now also U$52.P16; no longer U$52.P15
- net CAN2_TX: now also U$52.P17; no longer U$52.P16
- net GND: now also U$52.P2, U$53.P4, U$54.P2; no longer U$52.P1
- net I2C_SCL: now also U$52.P14, U$53.P2; no longer U$52.P13
- net I2C_SDA: now also U$52.P15, U$53.P3; no longer U$52.P14
- net UART4_RX: now also U$52.P11; no longer U$52.P10
- net UART4_TX: now also U$52.P10; no longer U$52.P9
- net USB_VBUS: now also U$57.P1
- net VBAT: now also U$58.2, U$59.2, U$60.2, U$62.2

Commit message: PCB ready for production
Parts:
- removed U$56: DIODE_SCHOTTKY, STM32F4:DIODE_SCHOTTKY
- added R13: 28, small_mavric:SMALL_MAVRIC_RESISTOR_R0402
- added U$63, U$64: PAD_FLASH, STM32F4:PAD_FLASH
- R14: value 28 -> 12.5
- U$54: value CON_2.54MM_2PINS_STACKABLE -> DIODE_SCHOTTKY; device STM32F4:CON_2.54MM_2PINS_STACKABLE -> STM32F4:DIODE_SCHOTTKY
- U$59: value 28 -> CON_2.54MM_2PINS; device small_mavric:SMALL_MAVRIC_RESISTOR_R0402 -> STM32F4:CON_2.54MM_2PINS
- renumbered U$10 to C20, U$12 to R17, U$13 to C22, U$14 to R18, U$15 to C6, U$16 to C5, U$17 to C4, U$18 to C3, U$19 to C2, U$20 to C1, U$21 to C9, U$22 to C10, U$23 to C14, U$24 to C15, U$25 to R7, U$26 to R6, U$27 to R4, U$28 to C7, U$3 to C16, U$30 to C11, U$32 to R1, U$33 to R5, U$34 to C8, U$35 to C13, U$36 to C12, U$37 to R3, U$38 to R16, U$39 to C23, U$44 to R8, U$45 to R9, U$46 to R10, U$47 to R11, U$48 to C24, U$49 to C25, U$5 to C18, U$50 to C26, U$51 to R2, U$58 to R12, U$6 to C17, U$60 to R15, U$62 to R14, U$8 to C19, U$9 to C21
Connections:
- removed net N$28: U$56.P2, U$59.1
- new net N$25: R15.1, U$54.P2
- new net SWCLK: U$1.PA14, U$63.P$1
- new net SWDIO: U$1.PA13, U$64.P$1
- net GND: now also U$59.P2; no longer U$54.P2
- net N$24: now also R13.1; no longer R14.1
- net N$29: now also R14.1; no longer R15.1
- net VBAT: now also R13.2; no longer U$59.2
- net VBAT_P: now also U$59.P1; no longer U$56.P1

Commit message: PCB finish with BOM
Parts:
- added U$3, U$5: PAD_FLASH, STM32F4:PAD_FLASH
Connections:
- net GND: now also U$3.P$1
- net VBAT: now also U$5.P$1
Changed lines of the file:
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@@
 <part name="U$63" library="STM32F4" deviceset="PAD_FLASH" device=""/>
 <part name="U$64" library="STM32F4" deviceset="PAD_FLASH" device=""/>
+<part name="U$3" library="STM32F4" deviceset="PAD_FLASH" device=""/>
+<part name="U$5" library="STM32F4" deviceset="PAD_FLASH" device=""/>
+<part name="GND24" library="supply1" deviceset="GND" device=""/>
 </parts>
 <sheets>
@@
 <instance part="U$63" gate="G$1" x="7.62" y="-27.94"/>
 <instance part="U$64" gate="G$1" x="7.62" y="-35.56"/>
+<instance part="U$3" gate="G$1" x="7.62" y="-43.18"/>
+<instance part="U$5" gate="G$1" x="7.62" y="-20.32"/>
+<instance part="GND24" gate="1" x="0" y="-45.72"/>
 </instances>
 <busses>
@@
 <pinref part="GND22" gate="1" pin="GND"/>
 </segment>
+<segment>
+<pinref part="U$3" gate="G$1" pin="P$1"/>
+<pinref part="GND24" gate="1" pin="GND"/>
+</segment>
 </net>
 <net name="USB_ID" class="0">
@@
 </segment>
 </net>
+<net name="VBAT" class="0">
+<segment>
+<pinref part="U$5" gate="G$1" pin="P$1"/>
+<wire x1="0" y1="-20.32" x2="-20.32" y2="-20.32" width="0.1524" layer="91"/>
+<label x="-17.78" y="-20.32" size="1.778" layer="95"/>
+</segment>
+</net>
